File: pcb/megadesk.kicad_sch (KiCad schematic)
At the start: 28 parts, among them J2 FFC, J3 AVR-ISP-6, J4 Interface, U1 7812, U2 HT7550-1, U3 ATtiny841-SS, U4 MCP2003B

Commit message: Add some component, change resistor value and change board size
Parts:
- added J1: Interface, Connector_PinHeader_2.54mm:PinHeader_1x05_P2.54mm_Horizontal, symbol Connector_Generic:Conn_01x05
- R1: value 1k -> 2k
Changed lines of the file:
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@@
 (kicad_sch
-	(version 20231120)
+	(version 20250114)
 	(generator "eeschema")
-	(generator_version "8.0")
+	(generator_version "9.0")
 	(paper "USLetter")
+	(text "Power Regulation"
+		(exclude_from_sim no)
+		(at 15.24 17.78 0)
+		(effects
+			(font
+				(size 1.524 1.524)
+			)
+			(justify left bottom)
+		)
+	)
+	(text "Headers"
+		(exclude_from_sim no)
+		(at 98.425 17.78 0)
+		(effects
+			(font
+				(size 1.3208 1.3208)
+			)
+			(justify left bottom)
+		)
+	)
+	(text "Volume control"
+		(exclude_from_sim no)
+		(at 152.4 104.14 0)
+		(effects
+			(font
+				(size 1.016 1.016)
+			)
+			(justify left bottom)
+		)
+	)
 	(junction
 		(at 218.44 77.47)
@@
 		)
 	)
-	(text "Power Regulation"
-		(exclude_from_sim no)
-		(at 15.24 17.78 0)
-		(effects
-			(font
-				(size 1.524 1.524)
-			)
-			(justify left bottom)
-		)
-	)
-	(text "Headers"
-		(exclude_from_sim no)
-		(at 98.425 17.78 0)
-		(effects
-			(font
-				(size 1.3208 1.3208)
-			)
-			(justify left bottom)
-		)
-	)
-	(text "Volume control"
-		(exclude_from_sim no)
-		(at 152.4 104.14 0)
-		(effects
-			(font
-				(size 1.016 1.016)
-			)
-			(justify left bottom)
-		)
-	)
 	(label "AVRRX"
 		(at 148.59 78.74 0)
-		(fields_autoplaced yes)
 		(effects
 			(font
@@
 	(label "MISO"
 		(at 130.81 81.28 0)
-		(fields_autoplaced yes)
 		(effects
 			(font
@@
 	(label "SCK"
 		(at 130.81 78.74 0)
-		(fields_autoplaced yes)
 		(effects
 			(font
@@
 	(label "RST"
 		(at 76.2 86.36 0)
-		(fields_autoplaced yes)
 		(effects
 			(font
@@
 	(label "AVRTX"
 		(at 148.59 81.28 0)
-		(fields_autoplaced yes)
 		(effects
 			(font
@@
 	(label "RST"
 		(at 134.62 99.06 0)
-		(fields_autoplaced yes)
 		(effects
 			(font
@@
 	(label "MOSI"
 		(at 130.81 83.82 0)
-		(fields_autoplaced yes)
 		(effects
 			(font
@@
 	(label "MISO"
 		(at 76.2 78.74 0)
-		(fields_autoplaced yes)
 		(effects
 			(font
@@
 	(label "AVRRX"
 		(at 119.38 33.02 180)
-		(fields_autoplaced yes)
 		(effects
 			(font
@@
 	(label "AVRTX"
 		(at 119.38 35.56 180)
-		(fields_autoplaced yes)
 		(effects
 			(font
@@
 	(label "MOSI"
 		(at 76.2 81.28 0)
-		(fields_autoplaced yes)
 		(effects
 			(font
@@
 	(label "SCK"
 		(at 76.2 83.82 0)
-		(fields_autoplaced yes)
 		(effects
 			(font
@@
 			)
 		)
-		(property "Value" "1k"
+		(property "Value" "2k"
 			(at 148.59 102.87 90)
 			(effects
@@
 	)
 	(symbol
+		(lib_id "Connector_Generic:Conn_01x05")
+		(at 109.22 134.62 0)
+		(unit 1)
+		(exclude_from_sim no)
+		(in_bom yes)
+		(on_board yes)
+		(dnp no)
+		(fields_autoplaced yes)
+		(property "Reference" "J1"
+			(at 111.76 133.985 0)
+			(effects
+				(font
+					(size 1.27 1.27)
+				)
+				(justify left)
+			)
+		)
+		(property "Value" "Interface"
+			(at 111.76 136.525 0)
+			(effects
+				(font
+					(size 1.27 1.27)
+				)
+				(justify left)
+			)
+		)
+		(property "Footprint" "Connector_PinHeader_2.54mm:PinHeader_1x05_P2.54mm_Horizontal"
+			(at 109.22 134.62 0)
+			(effects
+				(font
+					(size 1.27 1.27)
+				)
+				(hide yes)
+			)
+		)
+		(property "Datasheet" "~"
+			(at 109.22 134.62 0)
+			(effects
+				(font
+					(size 1.27 1.27)
+				)
+				(hide yes)
+			)
+		)
+		(property "Description" ""
+			(at 109.22 134.62 0)
+			(effects
+				(font
+					(size 1.27 1.27)
+				)
+				(hide yes)
+			)
+		)
+		(property "LCSC" "C492413"
+			(at 109.22 134.62 0)
+			(effects
+				(font
+					(size 1.27 1.27)
+				)
+				(hide yes)
+			)
+		)
+		(pin "1"
+		)
+		(pin "2"
+		)
+		(pin "3"
+		)
+		(pin "4"
+		)
+		(pin "5"
+		)
+		(instances
+			(project "megadesk"
+				(path "/457ea500-f3fa-4d58-b12b-1123e66fd2a7"
+					(reference "J1")
+					(unit 1)
+				)
+			)
+		)
+	)
+	(symbol
 		(lib_id "Connector:TestPoint")
 		(at 151.13 31.75 0)
@@
 		)
 	)
+	(embedded_fonts no)
 )
